Commit message: Add RGB-D camera simulation integration

File: src/robot_description/urdf/N1-Robot.urdf (robot description, URDF)
Before this commit: robot N1-Robot, 21 links, 20 joints
Links:
- added link dcw_depth_optical_frame
- added link dcw_rgbd_frame
- added link imu_frame
Joints:
- removed joint arm4_Joiint
- added joint arm4_Joint: type revolute, parent arm3, child arm4, origin xyz=0 0 0.08285 rpy=0 0 -0.027075, axis -2.6392E-05 -1 0, limit lower=-1.5708 upper=1.5708 effort=100 velocity=1
- added joint dcw_depth_optical_joint: type fixed, parent dcw_rgbd_frame, child dcw_depth_optical_frame, origin xyz=0 0 0 rpy=-1.5707963267949 0 -1.5707963267949
- added joint dcw_rgbd_joint: type fixed, parent DCW2, child dcw_rgbd_frame, origin xyz=0 0 0 rpy=0 0 0
- added joint imu_frame_joint: type fixed, parent base_link, child imu_frame, origin xyz=0.06 0 0.08 rpy=0 0 0
- joint Camera_Joint: axis 0 0 -1 -> (none); limit lower=0 upper=0 effort=0 velocity=0 -> (none); type revolute -> fixed
- joint llink1_Joint: mimic joint=rlink1_Joint multiplier=1 offset=0 -> (none)
- joint llink2_Joint: mimic joint=rlink1_Joint multiplier=-1 offset=0 -> (none)
- joint llink3_Joint: mimic joint=rlink1_Joint multiplier=1 offset=0 -> (none)
- joint lwheel1_Joint: limit lower=0 upper=0 effort=0 velocity=0 -> (none); type revolute -> continuous
- joint lwheel2_Joint: limit lower=0 upper=0 effort=0 velocity=0 -> (none); type revolute -> continuous
- joint rlink2_Joint: mimic joint=rlink1_Joint multiplier=1 offset=0 -> (none)
- joint rlink3_Joint: mimic joint=rlink1_Joint multiplier=-1 offset=0 -> (none)
- joint rwheel1_Joint: axis 0 0 -1 -> 0 0 1; limit lower=0 upper=0 effort=0 velocity=0 -> (none); type revolute -> continuous
- joint rwheel2_Joint: axis 0 0 -1 -> 0 0 1; limit lower=0 upper=0 effort=0 velocity=0 -> (none); type revolute -> continuous
