Commit message: add camera to the right arm add collison rule

File: src/piper_arm_description/urdf/piper_description.urdf.xacro (robot description, xacro)
@@ -8,12 +8,11 @@
     left_end_effector : none | gripper | revo2 | pika (왼쪽 arm)
     right_end_effector: none | gripper | revo2 | pika (오른쪽 arm)
-    with_camera_stand : true | false
-                        기본값: false; 왼쪽 gripper_base에 고정되는 카메라 스탠드를 로드합니다.
-    with_camera       : true | false
-                        기본값: false; RealSense D435 카메라를 로드합니다.
-                        주의: with_camera:=true에는 with_camera_stand:=true 설정이 필요합니다.
+    left_with_camera : true | false (기본값: false)
+    right_with_camera: true | false (기본값: false)
+                      해당 arm의 gripper_base에 카메라 스탠드와 D435를 로드합니다.
   사용 예시(명령줄에서 직접 파싱):
     xacro piper_description.urdf.xacro left_end_effector:=gripper right_end_effector:=pika
-    xacro piper_description.urdf.xacro with_camera_stand:=true with_camera:=true
+    xacro piper_description.urdf.xacro left_end_effector:=gripper left_with_camera:=true
+    xacro piper_description.urdf.xacro left_end_effector:=gripper right_end_effector:=gripper left_with_camera:=true right_with_camera:=true
 -->
 <robot xmlns:xacro="http://www.ros.org/wiki/xacro" name="piper">
@@ -25,8 +24,6 @@
   <!-- 두 arm base_link 사이의 Y축 간격(m) -->
   <xacro:arg name="arm_spacing"       default="0.60"/>
-  <!-- 카메라 스탠드 로드 여부; 기본값은 false입니다. -->
-  <xacro:arg name="with_camera_stand" default="false"/>
-  <!-- RealSense D435 로드 여부; 기본값은 false이며 with_camera_stand:=true가 필요합니다. -->
-  <xacro:arg name="with_camera"       default="false"/>
+  <xacro:arg name="left_with_camera"  default="false"/>
+  <xacro:arg name="right_with_camera" default="false"/>
   <!-- 조건식 평가를 위해 인자를 xacro 속성으로 변환합니다. -->
   <xacro:property name="left_ee"        value="$(arg left_end_effector)"/>
@@ -81,51 +78,53 @@
       <xacro:revo2_mount prefix="right_" parent="right_arm_link6" hand_base="right_base_link"/>
     </xacro:if>
-  <!-- ================================================================
-       카메라 스탠드(camera_stand_link)
-       with_camera_stand:=true일 때 로드
-       왼쪽 gripper_base에 고정
-       ================================================================ -->
-  <!-- Use xacro's boolean parser directly.  Storing "false" in a Python
-       expression would treat it as a non-empty (therefore truthy) string. -->
-  <xacro:if value="$(arg with_camera_stand)">
+  <!-- 두 카메라가 공유하는 재질과 센서 매크로는 한 번만 포함합니다. -->
+  <xacro:include filename="$(find realsense2_description)/urdf/_d435.urdf.xacro"/>
+  <!-- 각 gripper_base에 스탠드와 D435를 장착합니다. 왼쪽 링크 이름은 유지합니다. -->
+  <xacro:macro name="gripper_camera" params="prefix parent">
+      <link name="${prefix}camera_stand_link">
+        <inertial>
+          <origin rpy="0 0 0" xyz="0 0 0"/>
+          <mass value="0.2"/>
+          <inertia ixx="0.0002" ixy="0.0" ixz="0.0"
+                   iyy="0.0002" iyz="0.0"
+                   izz="0.0001"/>
+        </inertial>
+        <visual>
+          <origin rpy="-1.57 0 1.57" xyz="0 0 0"/>
+          <geometry>
+            <mesh filename="package://piper_arm_description/meshes/realsense_mid_stand.dae"/>
+          </geometry>
+        </visual>
+        <collision>
+          <origin rpy="0 0 0" xyz="0 0 0"/>
+          <geometry>
+            <mesh filename="package://piper_arm_description/meshes/realsense_mid_stand.dae"/>
+          </geometry>
+        </collision>
+      </link>
+      <joint name="${prefix}camera_stand_joint" type="fixed">
+        <origin xyz="-0.034 -0.001 0.022" rpy="0.0 0.0 0.0"/>
+        <parent link="${parent}"/>
+        <child link="${prefix}camera_stand_link"/>
+      </joint>
+      <link name="${prefix}d435_camera_link"/>
+      <joint name="${prefix}d435_camera_joint" type="fixed">
+        <origin xyz="-0.031 -0.028 0.0018" rpy="0.0 -1.22 0.0"/>
+        <parent link="${prefix}camera_stand_link"/>
+        <child link="${prefix}d435_camera_link"/>
+      </joint>
+      <xacro:sensor_d435 parent="${prefix}d435_camera_link" name="${prefix}camera">
+        <origin xyz="0 0 0" rpy="0 0 0"/>
+      </xacro:sensor_d435>
+  </xacro:macro>
+  <!-- xacro:if가 문자열 인자를 boolean으로 파싱합니다. -->
+  <xacro:if value="$(arg left_with_camera)">
     <xacro:if value="${left_ee == 'gripper'}">
-    <link name="camera_stand_link">
-      <inertial>
-        <origin rpy="0 0 0" xyz="0 0 0"/>
-        <mass value="0.2"/>
-        <inertia ixx="0.0002" ixy="0.0" ixz="0.0"
-                 iyy="0.0002" iyz="0.0"
-                 izz="0.0001"/>
-      </inertial>
-      <visual>
-        <origin rpy="-1.57 0 1.57" xyz="0 0 0"/>
-        <geometry>
-          <mesh filename="package://piper_arm_description/meshes/realsense_mid_stand.dae"/>
-        </geometry>
-      </visual>
-      <collision>
-        <origin rpy="0 0 0" xyz="0 0 0"/>
-        <geometry>
-          <mesh filename="package://piper_arm_description/meshes/realsense_mid_stand.dae"/>
-        </geometry>
-      </collision>
-    </link>
-    <joint name="camera_stand_joint" type="fixed">
-      <origin xyz="-0.034 -0.001 0.022" rpy="0.0 0.0 0.0"/>
-      <parent link="left_gripper_base"/>
-      <child link="camera_stand_link"/>
-    </joint>
+      <xacro:gripper_camera prefix="" parent="left_gripper_base"/>
     </xacro:if>
   </xacro:if>
-  <xacro:if value="$(arg with_camera_stand)">
-    <xacro:if value="$(arg with_camera)">
-      <xacro:if value="${left_ee == 'gripper'}">
-    <xacro:include filename="$(find realsense2_description)/urdf/test_d435_camera.urdf.xacro"/>
-    <joint name="d435_camera_joint" type="fixed">
-      <origin xyz="-0.031 -0.028 0.0018" rpy="0.0 -1.22 0.0"/>
-      <parent link="camera_stand_link"/>
-      <child link="d435_camera_link"/>
-    </joint>
-      </xacro:if>
+  <xacro:if value="$(arg right_with_camera)">
+    <xacro:if value="${right_ee == 'gripper'}">
+      <xacro:gripper_camera prefix="right_" parent="right_gripper_base"/>
     </xacro:if>
   </xacro:if>

File: src/piper_arm_moveit_config/config/piper_dual_gripper.urdf.xacro (robot description, xacro)
@@ -2,7 +2,7 @@
 <robot xmlns:xacro="http://www.ros.org/wiki/xacro" name="piper">
   <!-- The included description receives left/right_end_effector:=gripper from
-       the launch file.  Enable the D435 on the left gripper for this demo. -->
-  <xacro:arg name="with_camera_stand" default="true"/>
-  <xacro:arg name="with_camera" default="true"/>
+       the launch file. Enable a D435 on each gripper for this demo. -->
+  <xacro:arg name="left_with_camera" default="true"/>
+  <xacro:arg name="right_with_camera" default="true"/>
   <xacro:include filename="$(find piper_arm_description)/urdf/piper_description.urdf.xacro"/>
   <xacro:macro name="mock_joint" params="name initial:=0.0">

Commit message: add object add yolo redbox_detect

File: src/piper_arm_description/urdf/piper_description.urdf.xacro (robot description, xacro)
@@ -121,5 +121,5 @@
   <xacro:if value="$(arg left_with_camera)">
     <xacro:if value="${left_ee == 'gripper'}">
-      <xacro:gripper_camera prefix="" parent="left_gripper_base"/>
+      <xacro:gripper_camera prefix="left_" parent="left_gripper_base"/>
     </xacro:if>
   </xacro:if>

File: src/piper_arm_moveit_config/config/piper_dual_gripper.urdf.xacro (robot description, xacro)
@@ -22,4 +22,27 @@
       <state_interface name="velocity"><param name="initial_value">0.0</param></state_interface>
     </joint>
+  </xacro:macro>
+  <xacro:macro name="gazebo_rgbd_camera" params="prefix">
+    <gazebo reference="${prefix}camera_link">
+      <sensor name="${prefix}rgbd" type="rgbd_camera">
+        <pose>0 0 0 0 0 0</pose>
+        <gz_frame_id>${prefix}camera_link</gz_frame_id>
+        <always_on>true</always_on>
+        <update_rate>15</update_rate>
+        <topic>/${prefix}camera/rgbd</topic>
+        <camera>
+          <horizontal_fov>1.047</horizontal_fov>
+          <image>
+            <width>640</width>
+            <height>480</height>
+            <format>R8G8B8</format>
+          </image>
+          <clip>
+            <near>0.1</near>
+            <far>5.0</far>
+          </clip>
+        </camera>
+      </sensor>
+    </gazebo>
   </xacro:macro>
   <ros2_control name="PiperDualArmMockSystem" type="system">
@@ -47,4 +70,14 @@
       </plugin>
     </gazebo>
+    <xacro:if value="$(arg left_with_camera)">
+      <xacro:if value="${left_ee == 'gripper'}">
+        <xacro:gazebo_rgbd_camera prefix="left_"/>
+      </xacro:if>
+    </xacro:if>
+    <xacro:if value="$(arg right_with_camera)">
+      <xacro:if value="${right_ee == 'gripper'}">
+        <xacro:gazebo_rgbd_camera prefix="right_"/>
+      </xacro:if>
+    </xacro:if>
   </xacro:if>
 </robot>
